File: Schematics/KiCad Project/walkiepcb.kicad_pcb (KiCad board)
At the start: 2 copper layers, 45 x 100 mm, 87 parts, among them J1 USB-C / charge + program, J2 BAT+ / BAT-, J3 SW_PWR_IN / SW_PWR_OUT, J4 SPK+ / SPK-, J5 3V3 / POT_ADC / GND, J6 LED+ / LED-, J7 OLED MODULE: GND / 3V3 / SCL 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, Q1 MMBT3904, Q2 MMBT3904, Q3 FS8205A dual NMOS, Q4 AO3401A, SW1 BTN1 / hand-solder, SW2 BTN2 / hand-solder, SW3 BTN3 / hand-solder, SW4 BTN4 / hand-solder, SW5 BTN5 / hand-solder, U1 USBLC6-2SC6, U2 CH340C, U3 TP4056-42-ESOP8, U4 DW01A, U5 TPS63021DSJR, U6 ESP32-WROOM-32D-N16, U7 MAX98357AETE+T, U8 Ra-01SH / SX1262 915MHz

Commit message: Finalize BTN5 soft power PCB release
Parts:
- removed J3: SW_PWR_IN / SW_PWR_OUT, walkiepcb:WirePads_2_P5.08mm
- added D5: 1N4148WS, D_SOD-323, F.Cu at (37.0, 84.0)
- added D6: 1N4148WS, D_SOD-323, F.Cu at (35.0, 81.5)
- added Q5: AO3401A, SOT-23, F.Cu at (42.5, 70.7)
- added Q6: MMBT3904, SOT-23, F.Cu at (17.0, 6.00)
- added R27: 100k, R_0402_1005Metric, F.Cu at (44.0, 74.5)
- added R28: 100k, R_0402_1005Metric, F.Cu at (14.0, 3.00)
- added R30: 100k, R_0402_1005Metric, F.Cu at (17.5, 9.00)
- SW5: value BTN5 / hand-solder -> BTN5 POWER / FUNCTION
- TP8: value GPIO12 -> PWR_HOLD / GPIO12
- moved TP3 3.81 mm to (16.5, 13.5)
Connections:
- net /GPIO12 renamed /PWR_HOLD
- SW5 pad 1: /BTN5 -> /BTN5_SW
Routing:
- net /PWR_GATE: track 0.00 -> 130.3 mm, vias 0 -> 3
- net /PWR_LATCH_BASE: track 0.00 -> 17.6 mm
- net /USB_5V: track 173.4 -> 157.0 mm, vias 7 -> 9
- net /BTN5_SW: track 0.00 -> 7.81 mm
- net /SYS_FUSED: track 6.24 -> 11.2 mm, vias 1 -> 0
- net /BTN5: track 42.1 -> 45.1 mm, vias 1 -> 2
- net /UART_TX: track 71.2 -> 68.3 mm
- net /PWR_HOLD: track 65.5 -> 68.3 mm
- net /GND: track 490.8 -> 492.4 mm, vias 6 -> 8
- net /SYS_SW: track 108.3 -> 109.1 mm
Other:
- board text removed: "SYS_SW"
