File: Schematics/KiCad Project/walkiepcb.kicad_sch (KiCad schematic)
At the start: 83 parts, among them J1 USB-C / charge + program, J2 BAT+ / BAT-, J3 SW_PWR_IN / SW_PWR_OUT, J4 SPK+ / SPK-, J5 3V3 / POT_ADC / GND, J6 LED+ / LED-, J7 OLED MODULE: GND / 3V3 / SCL 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, Q1 MMBT3904, Q2 MMBT3904, Q3 FS8205A dual NMOS, Q4 AO3401A, SW1 BTN1 / hand-solder, SW2 BTN2 / hand-solder, SW3 BTN3 / hand-solder, SW4 BTN4 / hand-solder, SW5 BTN5 / hand-solder, U1 USBLC6-2SC6, U2 CH340C, U3 TP4056-42-ESOP8, U4 DW01A, U5 TPS63021DSJR, U6 ESP32-WROOM-32D-N16, U7 MAX98357AETE+T, U8 Ra-01SH / SX1262 915MHz

Commit message: Finalize BTN5 soft power PCB release
Parts:
- removed J3: SW_PWR_IN / SW_PWR_OUT, walkiepcb:WirePads_2_P5.08mm, symbol Connector_Generic:Conn_01x02
- added D5, D6: 1N4148WS, Diode_SMD:D_SOD-323, symbol Device:D_Schottky
- added Q5: AO3401A, Package_TO_SOT_SMD:SOT-23, symbol Transistor_FET:AO3401A
- added Q6: MMBT3904, Package_TO_SOT_SMD:SOT-23, symbol Transistor_BJT:Q_NPN_BEC
- added R27, R28, R30: 100k, Resistor_SMD:R_0402_1005Metric, symbol Device:R
- SW5: value BTN5 / hand-solder -> BTN5 POWER / FUNCTION; Notes Exactly two plated holes; ESP32 internal pull-up -> Hold 2 s for firmware-validated power on/off; pulls PWR_GAT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
- TP8: value GPIO12 -> PWR_HOLD / GPIO12; Notes Optional expansion solder/test pad -> Soft-power hold output and diagnostic pad; GPIO12 boot strap
Connections:
- net BTN5: now also D6.2 (A); no longer SW5.1
- net GND: now also Q6.3 (C), R28.2
- net SYS_FUSED: now also Q5.3 (D), R27.1
- net SYS_SW: now also Q5.2 (S)
- net GPIO12 renamed PWR_HOLD
- net PWR_HOLD: now also R30.1
- new net BTN5_SW: D5.1 (K), D6.1 (K), SW5.1
- new net PWR_GATE: D5.2 (A), Q5.1 (G), Q6.2 (E), R27.2
- new net PWR_LATCH_BASE: Q6.1 (B), R28.1, R30.2
Other:
- note added: "SOFT POWER: hold BTN5 for 2 s. A press immediately wakes hardware; firmware must assert GPIO12/PWR_HOLD only after validating the full 2 s startup hold. While running, release PWR_HOLD after a 2 s shutdown hold; power drops when BTN5 is released. Typical OFF leakage target <2 uA; verify prototypes over temperature."

Commit message: polishing
Parts:
- R1: footprint Resistor_SMD:R_0402_1005Metric -> Resistor_SMD:R_0603_1608Metric
Connections:
- net GND: now also Q6.2 (E); no longer Q6.3 (C)
- net PWR_GATE: now also Q6.3 (C); no longer Q6.2 (E)
- net SYS_FUSED: now also Q5.2 (S); no longer Q5.3 (D)
- net SYS_SW: now also Q5.3 (D); no longer Q5.2 (S)
Changed lines of the file:
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@@
 			)
 		)
-		(property "Footprint" "Resistor_SMD:R_0402_1005Metric"
+		(property "Footprint" "Resistor_SMD:R_0603_1608Metric"
 			(at 66.802 33.02 90)
 			(effects
@@
 		)
 	)
-	(label "SYS_FUSED"
+	(label "SYS_SW"
 		(at 304.80 132.08 90)
 		(effects
@@
 		)
 	)
-	(label "SYS_SW"
+	(label "SYS_FUSED"
 		(at 304.80 142.24 270)
 		(effects
@@
 		)
 	)
-	(label "GND"
+	(label "PWR_GATE"
 		(at 325.12 132.08 90)
 		(effects
@@
 		)
 	)
-	(label "PWR_GATE"
+	(label "GND"
 		(at 325.12 142.24 270)
 		(effects

Commit message: polishing
Parts:
- J5: value 3V3 / POT_ADC / GND -> POT
- TP8: value PWR_HOLD / GPIO12 -> GPIO12
- U3: value TP4056-42-ESOP8 -> TP4056
Connections:
- net 3V3: no longer J7.2 (Pin_2)
- net GND: no longer J7.1 (Pin_1)
- net OLED_SCL: no longer J7.3 (Pin_3)
- net OLED_SDA: no longer J7.4 (Pin_4)
- net SYS_SW: no longer C20.1
Other:
- note added: "BUCK BOOST"
- note added: "CELL PROTECTOR"
- note added: "ESP32"
- note added: "MIC, AMP"
- note added: "OLED HEADER"
- note added: "TP4056"
- note added: "USB UART"
- note added: "USB-C"
- note removed: "11–12 ESP32-WROOM MODULE, ADC, AND SX1262 RADIO"
- note removed: "13–15 I2S MICROPHONE, CLASS-D AMP, SPEAKER"
- note removed: "16 COMMERCIAL SSD1306 I2C OLED MODULE HEADER"
- note removed: "1–2 USB-C INPUT, CC SINK, AND ESD"
- note removed: "3–4 CH340C USB-UART / AUTO PROGRAM"
- note removed: "5 TP4056 CHARGER (~500 mA)"
- note removed: "6 CELL PROTECTION (DW01A + FS8205A)"
- note removed: "7–10 LOAD SHARE, PTC, SWITCH, 3.3 V BUCK-BOOST"
- note removed: "BAT_SENSE uses ADC1 GPIO1; POT_ADC uses ADC1 GPIO2. 100k/100k gives 4.2V -> 2.1V; 21uA drain. Firmware: warn about 3.3V and orderly shutdown about 3.0-3.1V loaded; DW01 cutoff is backup only."
- note removed: "Buttons: ESP32-S3 GPIO4/5/6/7/15 -> switch -> GND; firmware enables internal pull-ups. There are exactly 10 button holes, 3 pot holes, 2 LED holes, 4 OLED holes, and 2 power-switch holes."
- note removed: "Four through-hole connections only: pin 1 GND, pin 2 3V3, pin 3 SCL, pin 4 SDA. The commercial module supplies its own SSD1306 charge-pump parts; no raw SYS_SW reaches OLED logic."
- note removed: "GAIN_SLOT tied directly to GND = +12dB. GPIO4 high enables left-channel audio; low shuts down. MAX98357A raw supply sees ≈3.0–4.2V battery or ≈4.7V from USB after SS34 (<5.5V max)."
- note removed: "GPIO19/20 carry native USB D-/D+ through 22-ohm resistors. USB Serial/JTAG supports automatic download. VBUS is sensed through Q1 for self-powered USB-device firmware; this Type-C port remains a sink/device, not a host power source."
- note removed: "Overcurrent estimate: 150mV typical / (2×25mΩ) ≈3.0A at high gate; 150mV / (2×35mΩ) ≈2.14A at low gate. Tolerance/temp range is broader."
- note removed: "SOFT POWER: hold BTN5 for 2 s. A press immediately wakes hardware; firmware must assert GPIO12/PWR_HOLD only after validating the full 2 s startup hold. While running, release PWR_HOLD after a 2 s shutdown hold; power drops when BTN5 is released. Typical OFF leakage target <2 uA; verify prototypes over temperature."
- note removed: "USB present: D1 powers SYS_RAW and Q4 is off; TP4056 independently charges BAT_CELL. USB absent: Q4 body diode starts SYS_RAW then P-MOS turns on. Switch is downstream of charger. TPS63021 maintains 3.3V in buck/transition/boost; TI specifies 2A for VIN >2.5V. 2.2uH is sized for this <=1A rail."
- company: Custom design -> (none)
- title: ESP32 Walkie-Talkie — Economic PCBA schematic -> ESP32 Walkie-Talkie V2
- moved on the sheet: C15, C20, C29, J2, J7, Q3, Q5, R1, R19, R2
